Commit message: add trajectory

File: two_wheel_robot.urdf (robot description, URDF)
Before this commit: robot two_wheel_robot, 4 links, 3 joints
Joints:
- joint left_joint: origin xyz=0 0.1 -0.2 rpy=1.57079632679 0 0 -> xyz=0 0.1 -0.2 rpy=-1.57079632679 0 0
- joint right_joint: origin xyz=0 -0.1 -0.2 rpy=1.57079632679 0 0 -> xyz=0 -0.1 -0.2 rpy=-1.57079632679 0 0
